Commit message: Update diff_robot.urdf

File: merakm/urdf/diff_robot.urdf (robot description, URDF)
Before this commit: robot merakm, 7 links, 6 joints
Links:
- added link cam_link; visual box size=0.01 0.01 0.01
- link base_link: geometry visual box size=0.5 0.3 0.1
- link caster_wheel: geometry collision sphere radius=0.025; visual sphere radius=0.025
Joints:
- added joint cam_joint: type fixed, parent base_link, child cam_link, origin xyz=0.3 0.0 0.02 rpy=0.0 0.0 0.0
- joint base_lidar_joint: origin xyz=0.0 0.0 0.225 rpy=0.0 0.0 0.0 -> xyz=0.0 0.0 0.125 rpy=0.0 0.0 0.0
- joint caster_wheel_joint: origin xyz=0.2 0.0 -0.05 rpy=0.0 0.0 0.0 -> xyz=0.2 0.0 -0.07 rpy=0.0 0.0 0.0
- joint imu_joint: origin xyz=0.1 0.1 0.1 rpy=0.0 0.0 0.0 -> xyz=0.0 0.0 0.0 rpy=0.0 0.0 0.0
- joint left_wheel_joint: origin xyz=-0.175 0.225 0.0 rpy=0 0.0 0.0 -> xyz=-0.175 0.175 0.0 rpy=0 0.0 0.0
- joint right_wheel_joint: origin xyz=-0.175 -0.225 0.0 rpy=0 0.0 0.0 -> xyz=-0.175 -0.175 0.0 rpy=0 0.0 0.0

Commit message: Update diff_robot.urdf

File: merakm/urdf/diff_robot.urdf (robot description, URDF)
Before this commit: robot merakm, 8 links, 7 joints
Links:
- added link depth_link; visual box size=0.01 0.01 0.01
Joints:
- added joint depth_joint: type fixed, parent base_link, child depth_link, origin xyz=0.3 0.0 0.025 rpy=0.0 0.0 0.0

Commit message: Add files via upload

File: merakm/urdf/diff_robot.urdf (robot description, URDF)
Before this commit: robot merakm, 9 links, 8 joints
Links:
- removed link lidar_link
- added link base_scan, mass 0.114; collision cylinder length=0.05 radius=0.05; visual cylinder length=0.05 radius=0.1
Joints:
- removed joint base_lidar_joint
- added joint base_scan_joint: type fixed, parent base_link, child base_scan, origin xyz=0.0 0.0 0.125 rpy=0.0 0.0 0.0
- joint base_joint: child base_footprint -> base_link; parent base_link -> base_footprint
